Commit message: modified

File: install/robotiq_description/share/robotiq_description/urdf/robotiq_85_gripper.transmission.xacro (robot description, xacro)
@@ -1,41 +1,48 @@
 <?xml version="1.0"?>
-<robot xmlns:xacro="http://www.ros.org/wiki/xacro">
+<robot xmlns:xacro="http://ros.org/wiki/xacro">
   <xacro:macro name="robotiq_85_gripper_transmission" params="prefix">
-    <transmission name="${prefix}robotiq_85_left_knuckle_trans">
-      <type>transmission_interface/SimpleTransmission</type>
-      <joint name="${prefix}robotiq_85_left_knuckle_joint">
-        <hardwareInterface>PositionJointInterface</hardwareInterface>
-      </joint>
-      <actuator name="${prefix}robotiq_85_left_knuckle_motor">
-        <mechanicalReduction>1</mechanicalReduction>
-        <hardwareInterface>PositionJointInterface</hardwareInterface>
-      </actuator>
-    </transmission>
-    <gazebo>
-      <plugin filename="libgazebo_mimic_joint_plugin.so" name="${prefix}mimic_robotiq_85_1">
-        <joint>${prefix}robotiq_85_left_knuckle_joint</joint>
-        <mimicJoint>${prefix}robotiq_85_right_knuckle_joint</mimicJoint>
-      </plugin>
-      <plugin filename="libgazebo_mimic_joint_plugin.so" name="${prefix}mimic_robotiq_85_2">
-        <joint>${prefix}robotiq_85_left_knuckle_joint</joint>
-        <mimicJoint>${prefix}robotiq_85_left_inner_knuckle_joint</mimicJoint>
-      </plugin>
-      <plugin filename="libgazebo_mimic_joint_plugin.so" name="${prefix}mimic_robotiq_85_3">
-        <joint>${prefix}robotiq_85_left_knuckle_joint</joint>
-        <mimicJoint>${prefix}robotiq_85_right_inner_knuckle_joint</mimicJoint>
-      </plugin>
-      <plugin filename="libgazebo_mimic_joint_plugin.so" name="${prefix}mimic_robotiq_85_4">
-        <joint>${prefix}robotiq_85_left_knuckle_joint</joint>
-        <mimicJoint>${prefix}robotiq_85_left_finger_tip_joint</mimicJoint>
-        <multiplier>-1.0</multiplier>
-        <offset>0.0</offset>
-      </plugin>
-      <plugin filename="libgazebo_mimic_joint_plugin.so" name="${prefix}mimic_robotiq_85_5">
-        <joint>${prefix}robotiq_85_left_knuckle_joint</joint>
-        <mimicJoint>${prefix}robotiq_85_right_finger_tip_joint</mimicJoint>
-        <multiplier>-1.0</multiplier>
-        <offset>0.0</offset>
-      </plugin>
-    </gazebo>
-  </xacro:macro>
+        <transmission name="${prefix}robotiq_85_left_knuckle_trans">
+            <type>transmission_interface/SimpleTransmission</type>
+            <joint name="${prefix}robotiq_85_left_knuckle_joint">
+                <hardwareInterface>hardware_interface/PositionJointInterface</hardwareInterface>
+            </joint>
+            <actuator name="${prefix}robotiq_85_left_knuckle_motor">
+                <mechanicalReduction>1</mechanicalReduction>
+                <hardwareInterface>hardware_interface/PositionJointInterface</hardwareInterface>
+            </actuator>
+        </transmission>
+        <gazebo>
+                <!-- loading plugin: mimic joints works in gazebo now -->
+            <plugin filename="libroboticsgroup_gazebo_mimic_joint_plugin.so" name="${prefix}mimic_robotiq_85_1">
+                <joint>${prefix}robotiq_85_left_knuckle_joint</joint>
+                <mimicJoint>${prefix}robotiq_85_right_knuckle_joint</mimicJoint>
+                <!--multiplier>1.0</multiplier>
+                <offset>0.0</offset-->
+            </plugin>
+            <plugin filename="libroboticsgroup_gazebo_mimic_joint_plugin.so" name="${prefix}mimic_robotiq_85_2">
+                <joint>${prefix}robotiq_85_left_knuckle_joint</joint>
+                <mimicJoint>${prefix}robotiq_85_left_inner_knuckle_joint</mimicJoint>
+                <!--multiplier>1.0</multiplier>
+                <offset>0.0</offset-->
+            </plugin>
+            <plugin filename="libroboticsgroup_gazebo_mimic_joint_plugin.so" name="${prefix}mimic_robotiq_85_3">
+                <joint>${prefix}robotiq_85_left_knuckle_joint</joint>
+                <mimicJoint>${prefix}robotiq_85_right_inner_knuckle_joint</mimicJoint>
+                <!--multiplier>1.0</multiplier>
+                <offset>0.0</offset-->
+            </plugin>
+            <plugin filename="libroboticsgroup_gazebo_mimic_joint_plugin.so" name="${prefix}mimic_robotiq_85_4">
+                <joint>${prefix}robotiq_85_left_knuckle_joint</joint>
+                <mimicJoint>${prefix}robotiq_85_left_finger_tip_joint</mimicJoint>
+                <multiplier>-1.0</multiplier>
+                <offset>0.0</offset>
+            </plugin>
+            <plugin filename="libroboticsgroup_gazebo_mimic_joint_plugin.so" name="${prefix}mimic_robotiq_85_5">
+                <joint>${prefix}robotiq_85_left_knuckle_joint</joint>
+                <mimicJoint>${prefix}robotiq_85_right_finger_tip_joint</mimicJoint>
+                <multiplier>-1.0</multiplier>
+                <offset>0.0</offset>
+            </plugin>
+        </gazebo>
+    </xacro:macro>
 </robot>

File: install/ur5_robot_description/share/ur5_robot_description/urdf/ur5_gripper_main.xacro (robot description, xacro)
@@ -2,4 +2,7 @@
 <robot xmlns:xacro="http://www.ros.org/wiki/xacro" name="ur5_robot">
     <xacro:include filename="$(find ur5_robot_description)/urdf/eef.xacro"/>
+    <xacro:arg name="is_classic" default="true"/>
+    <xacro:include filename="$(find ur5_robot_description)/urdf/ur5_robot_gazebo.xacro"/>
+    <xacro:include filename="$(find ur5_robot_description)/urdf/ur5_ros2_control.xacro"/>
     <transmission name="shoulder_pan_trans">
         <type>transmission_interface/SimpleTransmission</type>
