Commit message: change korsi

File: install/robotiq_description/share/robotiq_description/urdf/robotiq_85_gripper.transmission.xacro (robot description, xacro)
@@ -1,48 +1,44 @@
 <?xml version="1.0"?>
-<robot xmlns:xacro="http://ros.org/wiki/xacro">
+<robot name="robotiq_85_gripper" xmlns:xacro="http://www.ros.org/wiki/xacro">
   <xacro:macro name="robotiq_85_gripper_transmission" params="prefix">
-        <transmission name="${prefix}robotiq_85_left_knuckle_trans">
-            <type>transmission_interface/SimpleTransmission</type>
-            <joint name="${prefix}robotiq_85_left_knuckle_joint">
-                <hardwareInterface>hardware_interface/PositionJointInterface</hardwareInterface>
-            </joint>
-            <actuator name="${prefix}robotiq_85_left_knuckle_motor">
-                <mechanicalReduction>1</mechanicalReduction>
-                <hardwareInterface>hardware_interface/PositionJointInterface</hardwareInterface>
-            </actuator>
-        </transmission>
-        <gazebo>
-                <!-- loading plugin: mimic joints works in gazebo now -->
-            <plugin filename="libroboticsgroup_gazebo_mimic_joint_plugin.so" name="${prefix}mimic_robotiq_85_1">
-                <joint>${prefix}robotiq_85_left_knuckle_joint</joint>
-                <mimicJoint>${prefix}robotiq_85_right_knuckle_joint</mimicJoint>
-                <!--multiplier>1.0</multiplier>
-                <offset>0.0</offset-->
-            </plugin>
-            <plugin filename="libroboticsgroup_gazebo_mimic_joint_plugin.so" name="${prefix}mimic_robotiq_85_2">
-                <joint>${prefix}robotiq_85_left_knuckle_joint</joint>
-                <mimicJoint>${prefix}robotiq_85_left_inner_knuckle_joint</mimicJoint>
-                <!--multiplier>1.0</multiplier>
-                <offset>0.0</offset-->
-            </plugin>
-            <plugin filename="libroboticsgroup_gazebo_mimic_joint_plugin.so" name="${prefix}mimic_robotiq_85_3">
-                <joint>${prefix}robotiq_85_left_knuckle_joint</joint>
-                <mimicJoint>${prefix}robotiq_85_right_inner_knuckle_joint</mimicJoint>
-                <!--multiplier>1.0</multiplier>
-                <offset>0.0</offset-->
-            </plugin>
-            <plugin filename="libroboticsgroup_gazebo_mimic_joint_plugin.so" name="${prefix}mimic_robotiq_85_4">
-                <joint>${prefix}robotiq_85_left_knuckle_joint</joint>
-                <mimicJoint>${prefix}robotiq_85_left_finger_tip_joint</mimicJoint>
-                <multiplier>-1.0</multiplier>
-                <offset>0.0</offset>
-            </plugin>
-            <plugin filename="libroboticsgroup_gazebo_mimic_joint_plugin.so" name="${prefix}mimic_robotiq_85_5">
-                <joint>${prefix}robotiq_85_left_knuckle_joint</joint>
-                <mimicJoint>${prefix}robotiq_85_right_finger_tip_joint</mimicJoint>
-                <multiplier>-1.0</multiplier>
-                <offset>0.0</offset>
-            </plugin>
-        </gazebo>
-    </xacro:macro>
+    <transmission name="${prefix}robotiq_85_left_knuckle_trans">
+      <type>transmission_interface/SimpleTransmission</type>
+      <joint name="${prefix}robotiq_85_left_knuckle_joint">
+        <hardwareInterface>PositionJointInterface</hardwareInterface>
+        <!-- <hardwareInterface>EffortJointInterface</hardwareInterface> -->
+      </joint>
+      <actuator name="${prefix}robotiq_85_left_knuckle_motor">
+        <mechanicalReduction>1</mechanicalReduction>
+        <hardwareInterface>PositionJointInterface</hardwareInterface>
+        <!-- <hardwareInterface>EfforJointInterface</hardwareInterface> -->
+      </actuator>
+    </transmission>
+    <!-- Mimic joints -->
+    <gazebo>
+      <plugin filename="libgazebo_mimic_joint_plugin.so" name="${prefix}mimic_robotiq_85_1">
+        <joint>${prefix}robotiq_85_left_knuckle_joint</joint>
+        <mimicJoint>${prefix}robotiq_85_right_knuckle_joint</mimicJoint>
+      </plugin>
+      <plugin filename="libgazebo_mimic_joint_plugin.so" name="${prefix}mimic_robotiq_85_2">
+        <joint>${prefix}robotiq_85_left_knuckle_joint</joint>
+        <mimicJoint>${prefix}robotiq_85_left_inner_knuckle_joint</mimicJoint>
+      </plugin>
+      <plugin filename="libgazebo_mimic_joint_plugin.so" name="${prefix}mimic_robotiq_85_3">
+        <joint>${prefix}robotiq_85_left_knuckle_joint</joint>
+        <mimicJoint>${prefix}robotiq_85_right_inner_knuckle_joint</mimicJoint>
+      </plugin>
+      <plugin filename="libgazebo_mimic_joint_plugin.so" name="${prefix}mimic_robotiq_85_4">
+        <joint>${prefix}robotiq_85_left_knuckle_joint</joint>
+        <mimicJoint>${prefix}robotiq_85_left_finger_tip_joint</mimicJoint>
+        <multiplier>-1.0</multiplier>
+        <offset>0.0</offset>
+      </plugin>
+      <plugin filename="libgazebo_mimic_joint_plugin.so" name="${prefix}mimic_robotiq_85_5">
+        <joint>${prefix}robotiq_85_left_knuckle_joint</joint>
+        <mimicJoint>${prefix}robotiq_85_right_finger_tip_joint</mimicJoint>
+        <multiplier>-1.0</multiplier>
+        <offset>0.0</offset>
+      </plugin>
+    </gazebo>
+  </xacro:macro>
 </robot>

File: install/robotiq_description/share/robotiq_description/urdf/robotiq_85_gripper.urdf.xacro (robot description, xacro)
@@ -53,6 +53,7 @@
                 </geometry>
             </collision>
-            <inertial>
-                <mass value="0.018491" />
+            <!--
+            <inertial>
+                <mass> 1.0 </mass>
                 <origin xyz="0.0 0.0 0.0" />
                 <inertia ixx = "0.000009" ixy = "-0.000001" ixz = "0.000000"
@@ -60,4 +61,20 @@
                          izx = "0.000000" izy = "0.000000" izz = "0.000010" />
             </inertial>
+            -->
+            <inertial>
+                    <!-- Volume:  6.8377110000e-06 -->
+                    <mass> 1.0 </mass>
+                    <!-- Center of mass:  9.2561000000e-04  0.0000000000e+00  1.7947540000e-02 -->
+                    <pose>  9.2561000000e-04  0.0000000000e+00  1.7947540000e-02 0 0 0 </pose>
+                    <!-- Inertia matrix -->
+                    <inertia>
+                        <ixx>  1.8679464517e-04 </ixx>
+                        <ixy> -1.4624777210e-11 </ixy>
+                        <ixz> -1.1207288521e-05 </ixz>
+                        <iyy>  2.0248142982e-04 </iyy>
+                        <iyz> -7.3123886049e-11 </iyz>
+                        <izz>  3.6687365114e-05 </izz>
+                    </inertia>
+            </inertial>
         </link>
         <link name="${prefix}robotiq_85_right_knuckle_link">
@@ -72,4 +89,5 @@
                 </geometry>
             </collision>
+            <!--
             <inertial>
                 <mass value="0.018491" />
@@ -78,4 +96,20 @@
                          iyx = "-0.000001" iyy = "0.000001" iyz = "0.000000"
                          izx = "0.000000" izy = "0.000000" izz = "0.000010" />
+            </inertial>
+            -->
+            <inertial>
+                    <!-- Volume:  6.8377110000e-06 -->
+                    <mass> 1.0 </mass>
+                    <!-- Center of mass:  9.2561000000e-04  0.0000000000e+00  1.7947540000e-02 -->
+                    <pose>  9.2561000000e-04  0.0000000000e+00  1.7947540000e-02 0 0 0 </pose>
+                    <!-- Inertia matrix -->
+                    <inertia>
+                        <ixx>  1.8679464517e-04 </ixx>
+                        <ixy> -1.4624777210e-11 </ixy>
+                        <ixz> -1.1207288521e-05 </ixz>
+                        <iyy>  2.0248142982e-04 </iyy>
+                        <iyz> -7.3123886049e-11 </iyz>
+                        <izz>  3.6687365114e-05 </izz>
+                    </inertia>
             </inertial>
         </link>
@@ -236,4 +270,19 @@
             </inertial>
         </link>
+        <!-- For better grasping-->
+        <gazebo reference="${prefix}robotiq_85_left_finger_tip_link">
+                    <kp>1000000.0</kp>
+                    <kd>1.0</kd>
+                    <mu1>1.0</mu1>
+                    <mu2>1.0</mu2>
+                    <minDepth>0.001</minDepth>
+        </gazebo>
+        <gazebo reference="${prefix}robotiq_85_right_finger_tip_link">
+                    <kp>1000000.0</kp>
+                    <kd>1.0</kd>
+                    <mu1>1.0</mu1>
+                    <mu2>1.0</mu2>
+                    <minDepth>0.001</minDepth>
+        </gazebo>
         <xacro:robotiq_85_gripper_transmission prefix="${prefix}" />
     </xacro:macro>

File: install/robotiq_description/share/robotiq_description/urdf/robotiq_85_gripper.xacro (robot description, xacro)
@@ -3,5 +3,5 @@
     <xacro:include filename="$(find robotiq_description)/urdf/robotiq_85_gripper.urdf.xacro" />
     <gazebo>
-        <plugin name="gazebo_ros_control" filename="libgazebo_ros_control.so">
+        <plugin filename="ign_ros2_control-system" name="ign_ros2_control::IgnitionROS2ControlPlugin">
             <robotNamespace>/robotiq_description</robotNamespace>
         </plugin>

File: install/robotiq_description/share/robotiq_description/urdf/robotiq_85_gripper2.xacro (robot description, xacro)
@@ -2,5 +2,5 @@
     <xacro:include filename="$(find robotiq_description)/urdf/robotiq_85_gripper.urdf.xacro" />
     <gazebo>
-        <plugin name="gazebo_ros_control" filename="libgazebo_ros_control.so">
+        <plugin name="ign_ros2_control::IgnitionROS2ControlPlugin" filename="ign_ros2_control-system">
             <robotNamespace>/robotiq_description</robotNamespace>
         </plugin>

File: install/ur5_robot_description/share/ur5_robot_description/urdf/ur5_gripper.xacro (robot description, xacro)
@@ -85,5 +85,4 @@
         </inertial>
     </link>
-    <!-- Fix the cobot to the world-->
     <link name="world"/>
     <joint name="fixed" type="fixed">
@@ -224,13 +223,7 @@
         </inertial>
     </link>
-    <!-- joints: main serial chain -->
     <joint name="base_link-base_link_inertia" type="fixed">
         <parent link="base_link" />
         <child link="base_link_inertia" />
-        <!-- 'base_link' is REP-103 aligned (so X+ forward), while the internal
-           frames of the robot/controller have X+ pointing backwards.
-           Use the joint between 'base_link' and 'base_link_inertia' (a dummy
-           link/frame) to introduce the necessary rotation over Z (of pi rad).
-      -->
         <origin rpy="0 0 3.141592653589793" xyz="0 0 0" />
     </joint>
@@ -311,5 +304,5 @@
     </joint>
     <gazebo>
-        <plugin name="gazebo_ros_control" filename="libgazebo_ros_control.so">
+        <plugin name="gazebo_ros_control" filename="ign_ros2_control-system">
             <robotNamespace>/ur5</robotNamespace>
         </plugin>

File: install/ur5_robot_description/share/ur5_robot_description/urdf/ur5_gripper_main.xacro (robot description, xacro)
@@ -5,64 +5,5 @@
     <xacro:include filename="$(find ur5_robot_description)/urdf/ur5_robot_gazebo.xacro"/>
     <xacro:include filename="$(find ur5_robot_description)/urdf/ur5_ros2_control.xacro"/>
-    <transmission name="shoulder_pan_trans">
-        <type>transmission_interface/SimpleTransmission</type>
-        <joint name="shoulder_pan_joint">
-            <hardwareInterface>hardware_interface/EffortJointInterface</hardwareInterface>
-        </joint>
-        <actuator name="shoulder_pan_motor">
-            <mechanicalReduction>1</mechanicalReduction>
-            <hardwareInterface>hardware_interface/EffortJointInterface</hardwareInterface>
-        </actuator>
-    </transmission>
-    <transmission name="shoulder_lift_trans">
-        <type>transmission_interface/SimpleTransmission</type>
-        <joint name="shoulder_lift_joint">
-            <hardwareInterface>hardware_interface/EffortJointInterface</hardwareInterface>
-        </joint>
-        <actuator name="shoulder_lift_motor">
-            <mechanicalReduction>1</mechanicalReduction>
-            <hardwareInterface>hardware_interface/EffortJointInterface</hardwareInterface>
-        </actuator>
-    </transmission>
-    <transmission name="elbow_trans">
-        <type>transmission_interface/SimpleTransmission</type>
-        <joint name="elbow_joint">
-            <hardwareInterface>hardware_interface/EffortJointInterface</hardwareInterface>
-        </joint>
-        <actuator name="elbow_motor">
-            <mechanicalReduction>1</mechanicalReduction>
-            <hardwareInterface>hardware_interface/EffortJointInterface</hardwareInterface>
-        </actuator>
-    </transmission>
-    <transmission name="wrist_1_trans">
-        <type>transmission_interface/SimpleTransmission</type>
-        <joint name="wrist_1_joint">
-            <hardwareInterface>hardware_interface/EffortJointInterface</hardwareInterface>
-        </joint>
-        <actuator name="wrist_1_motor">
-            <mechanicalReduction>1</mechanicalReduction>
-            <hardwareInterface>hardware_interface/EffortJointInterface</hardwareInterface>
-        </actuator>
-    </transmission>
-    <transmission name="wrist_2_trans">
-        <type>transmission_interface/SimpleTransmission</type>
-        <joint name="wrist_2_joint">
-            <hardwareInterface>hardware_interface/EffortJointInterface</hardwareInterface>
-        </joint>
-        <actuator name="wrist_2_motor">
-            <mechanicalReduction>1</mechanicalReduction>
-            <hardwareInterface>hardware_interface/EffortJointInterface</hardwareInterface>
-        </actuator>
-    </transmission>
-    <transmission name="wrist_3_trans">
-        <type>transmission_interface/SimpleTransmission</type>
-        <joint name="wrist_3_joint">
-            <hardwareInterface>hardware_interface/EffortJointInterface</hardwareInterface>
-        </joint>
-        <actuator name="wrist_3_motor">
-            <mechanicalReduction>1</mechanicalReduction>
-            <hardwareInterface>hardware_interface/EffortJointInterface</hardwareInterface>
-        </actuator>
-    </transmission>
+    <xacro:include filename="$(find ur5_robot_description)/urdf/ur5_robot_transmission.xacro"/>
     <link name="base_link" />
     <link name="base_link_inertia">
@@ -70,5 +11,5 @@
             <origin rpy="0 0 3.141592653589793" xyz="0 0 0" />
             <geometry>
-                <mesh filename="package://ur5_robot_description/meshes/base.dae" />
+                <mesh filename="package://ur5_robot_description/meshes/visual/base.dae" />
             </geometry>
             <material name="LightGrey">
@@ -98,5 +39,5 @@
             <origin rpy="0 0 3.141592653589793" xyz="0 0 0" />
             <geometry>
-                <mesh filename="package://ur5_robot_description/meshes/shoulder.dae" />
+                <mesh filename="package://ur5_robot_description/meshes/visual/shoulder.dae" />
             </geometry>
             <material name="LightGrey">
@@ -120,5 +61,5 @@
             <origin rpy="1.5707963267948966 0 -1.5707963267948966" xyz="0 0 0.13585" />
             <geometry>
-                <mesh filename="package://ur5_robot_description/meshes/upperarm.dae" />
+                <mesh filename="package://ur5_robot_description/meshes/visual/upperarm.dae" />
             </geometry>
             <material name="LightGrey">
@@ -142,5 +83,5 @@
             <origin rpy="1.5707963267948966 0 -1.5707963267948966" xyz="0 0 0.0165" />
             <geometry>
-                <mesh filename="package://ur5_robot_description/meshes/forearm.dae" />
+                <mesh filename="package://ur5_robot_description/meshes/visual/forearm.dae" />
             </geometry>
             <material name="LightGrey">
@@ -164,5 +105,5 @@
             <origin rpy="1.5707963267948966 0 0" xyz="0 0 -0.093" />
             <geometry>
-                <mesh filename="package://ur5_robot_description/meshes/wrist1.dae" />
+                <mesh filename="package://ur5_robot_description/meshes/visual/wrist1.dae" />
             </geometry>
             <material name="LightGrey">
@@ -186,5 +127,5 @@
             <origin rpy="0 0 0" xyz="0 0 -0.095" />
             <geometry>
-                <mesh filename="package://ur5_robot_description/meshes/wrist2.dae" />
+                <mesh filename="package://ur5_robot_description/meshes/visual/wrist2.dae" />
             </geometry>
             <material name="LightGrey">
@@ -208,5 +149,5 @@
             <origin rpy="1.5707963267948966 0 0" xyz="0 0 -0.0818" />
             <geometry>
-                <mesh filename="package://ur5_robot_description/meshes/wrist3.dae" />
+                <mesh filename="package://ur5_robot_description/meshes/visual/wrist3.dae" />
             </geometry>
             <material name="LightGrey">
@@ -298,5 +239,5 @@
     </joint>
     <gazebo>
-        <plugin name="gazebo_ros_control" filename="libgazebo_ros_control.so">
+        <plugin filename="ign_ros2_control-system" name="ign_ros2_control::IgnitionROS2ControlPlugin">
             <robotNamespace>/ur5</robotNamespace>
         </plugin>

File: install/ur5_robot_description/share/ur5_robot_description/urdf/ur5_robot_gazebo.xacro (robot description, xacro)
@@ -2,14 +2,16 @@
 <robot xmlns:xacro="http://www.ros.org/wiki/xacro" name="ur5_robot">
    <gazebo>
-     <xacro:if value="$(arg is_classic)">
-       <plugin filename="gz_ros2_control-system" name="gz_ros2_control::GazeboSimROS2ControlPlugin">
-         <parameters>$(find ur5_controller)/config/ur5_controller.yaml</parameters>
-       </plugin>
-     </xacro:if>
-     <xacro:unless value="$(arg is_classic)">
-       <plugin filename="ign_ros2_control-system" name="ign_ros2_control::IgnitionROS2ControlPlugin">
-         <parameters>$(find ur5_controller)/config/ur5_controller.yaml</parameters>
-       </plugin>
-     </xacro:unless>
-   </gazebo>
+    <!-- ROS 2 Humble -->
+    <xacro:if value="$(arg is_classic)">
+      <plugin filename="libign_ros2_control-system.so" name="ign_ros2_control::IgnitionROS2ControlPlugin">
+        <parameters>$(find ur5_controller)/config/ur5_controller.yaml</parameters>
+      </plugin>
+    </xacro:if>
+    <!-- ROS 2 Iron or above -->
+    <xacro:unless value="$(arg is_classic)">
+      <plugin filename="libgazebo_ros2_control.so" name="gazebo_ros2_control">
+        <parameters>$(find ur5_controller)/config/ur5_controller.yaml</parameters>
+      </plugin>
+    </xacro:unless>
+  </gazebo>
 </robot>
