Commit message: change korsi

File: install/ur5_robot_description/share/ur5_robot_description/urdf/ur5_ros2_control.xacro (robot description, xacro)
@@ -1,32 +1,16 @@
 <?xml version="1.0" ?>
 <robot xmlns:xacro="http://www.ros.org/wiki/xacro" name="ur5_robot">
- <xacro:macro name="ur_ros2_control" params="
-    name
-    prefix
-    use_fake_hardware:=false fake_sensor_commands:=false
-    sim_gazebo:=false
-    sim_ignition:=false
-    headless_mode:=false
-    initial_positions:=${dict(shoulder_pan_joint=0.0,shoulder_lift_joint=-1.57,elbow_joint=0.0,wrist_1_joint=-1.57,wrist_2_joint=0.0,wrist_3_joint=0.0)}
-    use_tool_communication:=false
-    script_filename output_recipe_filename
-    input_recipe_filename tf_prefix
-    hash_kinematics robot_ip
-    tool_voltage:=24 tool_parity:=0 tool_baud_rate:=115200 tool_stop_bits:=1
-    tool_rx_idle_chars:=1.5 tool_tx_idle_chars:=3.5 tool_device_name:=/tmp/ttyUR tool_tcp_port:=54321
-    reverse_port:=50001
-    script_sender_port:=50002">
 <ros2_control type="system" name="RobotSystem">
    <xacro:if value="$(arg is_classic)">
      <hardware>
-       <plugin>gz_ros2_control/GazeboSimSystem</plugin>
+       <plugin>ign_ros2_control/IgnitionSystem</plugin>
      </hardware>
    </xacro:if>
    <xacro:unless value="$(arg is_classic)">
      <hardware>
-       <plugin>ign_ros2_control/IgnitionSystem</plugin>
+       <plugin>gz_ros2_control/GazeboSimSystem</plugin>
      </hardware>
    </xacro:unless>
- <joint name="${prefix}shoulder_pan_joint">
+ <joint name="shoulder_pan_joint">
         <command_interface name="position">
           <param name="min">{-2*pi}</param>
@@ -38,10 +22,10 @@
         </command_interface>
         <state_interface name="position">
-          <param name="initial_value">${initial_positions['shoulder_pan_joint']}</param>
+          <param name="initial_value">0.0</param>
         </state_interface>
         <state_interface name="velocity"/>
         <state_interface name="effort"/>
  </joint>
- <joint name="${prefix}shoulder_lift_joint">
+ <joint name="shoulder_lift_joint">
         <command_interface name="position">
           <param name="min">{-2*pi}</param>
@@ -54,10 +38,10 @@
         <state_interface name="position">
           <!-- initial position for the FakeSystem and simulation -->
-          <param name="initial_value">${initial_positions['shoulder_lift_joint']}</param>
+          <param name="initial_value">-1.57</param>
         </state_interface>
         <state_interface name="velocity"/>
         <state_interface name="effort"/>
   </joint>
-   <joint name="${prefix}elbow_joint">
+   <joint name="elbow_joint">
         <command_interface name="position">
           <param name="min">{-pi}</param>
@@ -70,10 +54,10 @@
         <state_interface name="position">
           <!-- initial position for the FakeSystem and simulation -->
-          <param name="initial_value">${initial_positions['elbow_joint']}</param>
+          <param name="initial_value">0.0</param>
         </state_interface>
         <state_interface name="velocity"/>
         <state_interface name="effort"/>
     </joint>
-    <joint name="${prefix}wrist_1_joint">
+    <joint name="wrist_1_joint">
         <command_interface name="position">
           <param name="min">{-2*pi}</param>
@@ -86,10 +70,10 @@
         <state_interface name="position">
           <!-- initial position for the FakeSystem and simulation -->
-          <param name="initial_value">${initial_positions['wrist_1_joint']}</param>
+          <param name="initial_value">-1.57</param>
         </state_interface>
         <state_interface name="velocity"/>
         <state_interface name="effort"/>
     </joint>
-    <joint name="${prefix}wrist_2_joint">
+    <joint name="wrist_2_joint">
         <command_interface name="position">
           <param name="min">{-2*pi}</param>
@@ -102,10 +86,10 @@
         <state_interface name="position">
           <!-- initial position for the FakeSystem and simulation -->
-          <param name="initial_value">${initial_positions['wrist_2_joint']}</param>
+          <param name="initial_value">0.0</param>
         </state_interface>
         <state_interface name="velocity"/>
         <state_interface name="effort"/>
     </joint>
-    <joint name="${prefix}wrist_3_joint">
+    <joint name="wrist_3_joint">
         <command_interface name="position">
           <param name="min">{-2*pi}</param>
@@ -118,5 +102,5 @@
         <state_interface name="position">
           <!-- initial position for the FakeSystem and simulation -->
-          <param name="initial_value">${initial_positions['wrist_3_joint']}</param>
+          <param name="initial_value">0.0</param>
         </state_interface>
         <state_interface name="velocity"/>
@@ -166,4 +150,3 @@
     </joint>
 </ros2_control>
- </xacro:macro>
 </robot>

Commit message: changes made

File: install/robotiq_description/share/robotiq_description/urdf/robotiq_85_gripper.transmission.xacro (robot description, xacro)
@@ -14,31 +14,4 @@
       </actuator>
     </transmission>
-    <!-- Mimic joints -->
-    <gazebo>
-      <plugin filename="libgazebo_mimic_joint_plugin.so" name="${prefix}mimic_robotiq_85_1">
-        <joint>${prefix}robotiq_85_left_knuckle_joint</joint>
-        <mimicJoint>${prefix}robotiq_85_right_knuckle_joint</mimicJoint>
-      </plugin>
-      <plugin filename="libgazebo_mimic_joint_plugin.so" name="${prefix}mimic_robotiq_85_2">
-        <joint>${prefix}robotiq_85_left_knuckle_joint</joint>
-        <mimicJoint>${prefix}robotiq_85_left_inner_knuckle_joint</mimicJoint>
-      </plugin>
-      <plugin filename="libgazebo_mimic_joint_plugin.so" name="${prefix}mimic_robotiq_85_3">
-        <joint>${prefix}robotiq_85_left_knuckle_joint</joint>
-        <mimicJoint>${prefix}robotiq_85_right_inner_knuckle_joint</mimicJoint>
-      </plugin>
-      <plugin filename="libgazebo_mimic_joint_plugin.so" name="${prefix}mimic_robotiq_85_4">
-        <joint>${prefix}robotiq_85_left_knuckle_joint</joint>
-        <mimicJoint>${prefix}robotiq_85_left_finger_tip_joint</mimicJoint>
-        <multiplier>-1.0</multiplier>
-        <offset>0.0</offset>
-      </plugin>
-      <plugin filename="libgazebo_mimic_joint_plugin.so" name="${prefix}mimic_robotiq_85_5">
-        <joint>${prefix}robotiq_85_left_knuckle_joint</joint>
-        <mimicJoint>${prefix}robotiq_85_right_finger_tip_joint</mimicJoint>
-        <multiplier>-1.0</multiplier>
-        <offset>0.0</offset>
-      </plugin>
-    </gazebo>
   </xacro:macro>
 </robot>

File: install/robotiq_description/share/robotiq_description/urdf/robotiq_85_gripper.urdf.xacro (robot description, xacro)
@@ -53,27 +53,17 @@
                 </geometry>
             </collision>
-            <!--
-            <inertial>
-                <mass> 1.0 </mass>
-                <origin xyz="0.0 0.0 0.0" />
-                <inertia ixx = "0.000009" ixy = "-0.000001" ixz = "0.000000"
-                         iyx = "-0.000001" iyy = "0.000001" iyz = "0.000000"
-                         izx = "0.000000" izy = "0.000000" izz = "0.000010" />
-            </inertial>
-            -->
-            <inertial>
-                    <!-- Volume:  6.8377110000e-06 -->
-                    <mass> 1.0 </mass>
-                    <!-- Center of mass:  9.2561000000e-04  0.0000000000e+00  1.7947540000e-02 -->
-                    <pose>  9.2561000000e-04  0.0000000000e+00  1.7947540000e-02 0 0 0 </pose>
-                    <!-- Inertia matrix -->
-                    <inertia>
-                        <ixx>  1.8679464517e-04 </ixx>
-                        <ixy> -1.4624777210e-11 </ixy>
-                        <ixz> -1.1207288521e-05 </ixz>
-                        <iyy>  2.0248142982e-04 </iyy>
-                        <iyz> -7.3123886049e-11 </iyz>
-                        <izz>  3.6687365114e-05 </izz>
-                    </inertia>
+            <inertial>
+                <origin
+                        xyz="0.0178331863169983 3.68915177224286E-11 0.0021442477325704"
+                        rpy="0 0 0" />
+                <mass
+                        value="0.00684838849434396" />
+                <inertia
+                        ixx="2.66832029033166E-07"
+                        ixy="1.66142314639824E-15"
+                        ixz="1.45945633322873E-07"
+                        iyy="1.3889233257419E-06"
+                        iyz="2.82951161241588E-15"
+                        izz="1.26603336914415E-06" />
             </inertial>
         </link>
@@ -89,27 +79,17 @@
                 </geometry>
             </collision>
-            <!--
-            <inertial>
-                <mass value="0.018491" />
-                <origin xyz="0.0 0.0 0.0" />
-                <inertia ixx = "0.000009" ixy = "-0.000001" ixz = "0.000000"
-                         iyx = "-0.000001" iyy = "0.000001" iyz = "0.000000"
-                         izx = "0.000000" izy = "0.000000" izz = "0.000010" />
-            </inertial>
-            -->
-            <inertial>
-                    <!-- Volume:  6.8377110000e-06 -->
-                    <mass> 1.0 </mass>
-                    <!-- Center of mass:  9.2561000000e-04  0.0000000000e+00  1.7947540000e-02 -->
-                    <pose>  9.2561000000e-04  0.0000000000e+00  1.7947540000e-02 0 0 0 </pose>
-                    <!-- Inertia matrix -->
-                    <inertia>
-                        <ixx>  1.8679464517e-04 </ixx>
-                        <ixy> -1.4624777210e-11 </ixy>
-                        <ixz> -1.1207288521e-05 </ixz>
-                        <iyy>  2.0248142982e-04 </iyy>
-                        <iyz> -7.3123886049e-11 </iyz>
-                        <izz>  3.6687365114e-05 </izz>
-                    </inertia>
+            <inertial>
+                <origin
+                    xyz="0.0168606186773776 3.93808471820465E-10 0.0226699950793434"
+                    rpy="0 0 0" />
+                <mass
+                    value="0.0110930853895903" />
+                <inertia
+                    ixx="4.27134775939882E-06"
+                    ixy="-8.53568456728898E-15"
+                    ixz="1.77774229944246E-06"
+                    iyy="3.96548790524392E-06"
+                    iyz="-8.45108024914164E-15"
+                    izz="3.20325997634666E-06" />
             </inertial>
         </link>

File: install/ur5_robot_description/share/ur5_robot_description/urdf/ur5_robot_gazebo.xacro (robot description, xacro)
@@ -4,5 +4,5 @@
     <!-- ROS 2 Humble -->
     <xacro:if value="$(arg is_classic)">
-      <plugin filename="libign_ros2_control-system.so" name="ign_ros2_control::IgnitionROS2ControlPlugin">
+      <plugin filename="ign_ros2_control-system" name="ign_ros2_control::IgnitionROS2ControlPlugin">
         <parameters>$(find ur5_controller)/config/ur5_controller.yaml</parameters>
       </plugin>
@@ -10,5 +10,5 @@
     <!-- ROS 2 Iron or above -->
     <xacro:unless value="$(arg is_classic)">
-      <plugin filename="libgazebo_ros2_control.so" name="gazebo_ros2_control">
+      <plugin filename="gz_ros2_control-system" name="gz_ros2_control::GazeboSimROS2ControlPlugin">
         <parameters>$(find ur5_controller)/config/ur5_controller.yaml</parameters>
       </plugin>

File: install/ur5_robot_description/share/ur5_robot_description/urdf/ur5_ros2_control.xacro (robot description, xacro)
@@ -4,11 +4,11 @@
    <xacro:if value="$(arg is_classic)">
      <hardware>
-       <plugin>ign_ros2_control/IgnitionSystem</plugin>
-     </hardware>
+        <plugin>ign_ros2_control/IgnitionSystem</plugin>
+      </hardware>
    </xacro:if>
    <xacro:unless value="$(arg is_classic)">
      <hardware>
-       <plugin>gz_ros2_control/GazeboSimSystem</plugin>
-     </hardware>
+        <plugin>gz_ros2_control/GazeboSimSystem</plugin>
+      </hardware>
    </xacro:unless>
  <joint name="shoulder_pan_joint">
@@ -16,8 +16,4 @@
           <param name="min">{-2*pi}</param>
           <param name="max">{2*pi}</param>
-        </command_interface>
-        <command_interface name="velocity">
-          <param name="min">-3.15</param>
-          <param name="max">3.15</param>
         </command_interface>
         <state_interface name="position">
@@ -31,8 +27,4 @@
           <param name="min">{-2*pi}</param>
           <param name="max">{2*pi}</param>
-        </command_interface>
-        <command_interface name="velocity">
-          <param name="min">-3.15</param>
-          <param name="max">3.15</param>
         </command_interface>
         <state_interface name="position">
@@ -48,8 +40,4 @@
           <param name="max">{pi}</param>
         </command_interface>
-        <command_interface name="velocity">
-          <param name="min">-3.15</param>
-          <param name="max">3.15</param>
-        </command_interface>
         <state_interface name="position">
           <!-- initial position for the FakeSystem and simulation -->
@@ -63,8 +51,4 @@
           <param name="min">{-2*pi}</param>
           <param name="max">{2*pi}</param>
-        </command_interface>
-        <command_interface name="velocity">
-          <param name="min">-3.2</param>
-          <param name="max">3.2</param>
         </command_interface>
         <state_interface name="position">
@@ -80,8 +64,4 @@
           <param name="max">{2*pi}</param>
         </command_interface>
-        <command_interface name="velocity">
-          <param name="min">-3.2</param>
-          <param name="max">3.2</param>
-        </command_interface>
         <state_interface name="position">
           <!-- initial position for the FakeSystem and simulation -->
@@ -95,8 +75,4 @@
           <param name="min">{-2*pi}</param>
           <param name="max">{2*pi}</param>
-        </command_interface>
-        <command_interface name="velocity">
-          <param name="min">-3.2</param>
-          <param name="max">3.2</param>
         </command_interface>
         <state_interface name="position">

File: src/ur5_robot_description/urdf/ur5_gripper_main.xacro (robot description, xacro)
@@ -240,5 +240,5 @@
     <gazebo>
         <plugin filename="ign_ros2_control-system" name="ign_ros2_control::IgnitionROS2ControlPlugin">
-            <robotNamespace>/ur5</robotNamespace>
+            <robotNamespace>/controller_manager</robotNamespace>
         </plugin>
     </gazebo>
