Commit message: abar change korsi

File: install/robotiq_description/share/robotiq_description/urdf/robotiq_85_gripper.urdf.xacro (robot description, xacro)
@@ -55,5 +55,5 @@
           <parent link="robotiq_85_base_link"/>
           <child  link="camera_link"/>
-          <origin xyz="0.052 0 0.02" rpy="0 0 0"/>
+          <origin xyz="0.020 0 0.044" rpy="${pi/2} 0 ${pi/2}"/>
         </joint>
         <joint name="camera_link_to_camera_frame_link" type="fixed">
@@ -129,10 +129,10 @@
             </inertial>
         </link>
-        <joint name="${prefix}robotiq_85_left_finger_joint" type="fixed">
+        <joint name="${prefix}robotiq_85_left_finger_joint" type="continuous">
             <parent link="${prefix}robotiq_85_left_knuckle_link"/>
             <child link="${prefix}robotiq_85_left_finger_link"/>
             <origin xyz="-0.00408552455 -0.03148604435 0.0" rpy="0 0 0" />
         </joint>
-        <joint name="${prefix}robotiq_85_right_finger_joint" type="fixed">
+        <joint name="${prefix}robotiq_85_right_finger_joint" type="continuous">
             <parent link="${prefix}robotiq_85_right_knuckle_link"/>
             <child link="${prefix}robotiq_85_right_finger_link"/>

File: install/ur5_gripper_moveit_config/share/ur5_gripper_moveit_config/config/ur5_robot.urdf.xacro (robot description, xacro)
@@ -6,4 +6,4 @@
     <!-- Import control_xacro -->
     <xacro:include filename="ur5_robot.ros2_control.xacro" />
-    <xacro:ur5_robot_ros2_control name="FakeSystem" initial_positions_file="$(arg initial_positions_file)"/>
+    <xacro:ur5_robot_ros2_control name="RobotSystem" initial_positions_file="$(arg initial_positions_file)"/>
 </robot>

File: install/ur5_robot_description/share/ur5_robot_description/urdf/ur5_ros2_control.xacro (robot description, xacro)
@@ -85,6 +85,6 @@
     <!--gripper control-->
     <joint name="robotiq_85_left_knuckle_joint">
-                <param name="initial_position">0.7929</param>
-                <command_interface name="position" />
+                <param name="initial_position">0</param>
+                <command_interface name="position"/>
                 <state_interface name="position"/>
                 <state_interface name="velocity"/>
@@ -125,8 +125,6 @@
                 <state_interface name="velocity"/>
     </joint>
-    <!--
     <joint name="robotiq_85_left_finger_joint">
-                <param name="mimic">robotiq_85_left_knuckle_joint</param>
-                <param name="multiplier">1</param>
+                <param name="initial_position">0</param>
                 <command_interface name="position" />
                 <state_interface name="position"/>
@@ -134,11 +132,9 @@
     </joint>
     <joint name="robotiq_85_right_finger_joint">
-                <param name="mimic">robotiq_85_left_knuckle_joint</param>
-                <param name="multiplier">-1</param>
+                <param name="initial_position">0</param>
                 <command_interface name="position" />
                 <state_interface name="position"/>
                 <state_interface name="velocity"/>
     </joint>
-    -->
 </ros2_control>
 </robot>

File: src/ur5_robot_description/urdf/ur5_ros2_control.xacro (robot description, xacro)
@@ -85,6 +85,6 @@
     <!--gripper control-->
     <joint name="robotiq_85_left_knuckle_joint">
-                <param name="initial_position">0.7929</param>
-                <command_interface name="position" />
+                <param name="initial_position">0</param>
+                <command_interface name="position"/>
                 <state_interface name="position"/>
                 <state_interface name="velocity"/>
@@ -126,6 +126,5 @@
     </joint>
     <joint name="robotiq_85_left_finger_joint">
-                <param name="mimic">robotiq_85_left_knuckle_joint</param>
-                <param name="multiplier">1</param>
+                <param name="initial_position">0</param>
                 <command_interface name="position" />
                 <state_interface name="position"/>
@@ -133,6 +132,5 @@
     </joint>
     <joint name="robotiq_85_right_finger_joint">
-                <param name="mimic">robotiq_85_left_knuckle_joint</param>
-                <param name="multiplier">-1</param>
+                <param name="initial_position">0</param>
                 <command_interface name="position" />
                 <state_interface name="position"/>
